File: BusPlate/BusPlate.kicad_pcb (KiCad board)
At the start: 4 copper layers, 46 x 46 mm, 48 parts, among them J1 USB_C_Receptacle_USB2.0_14P, J12 RJ45, J13 RJ45, J2 Conn_01x16_Pin, SW1 SW_Push, SW2 SW_DIP_x01, U1 RP2040, U2 MCP1700x-330xxMB, U3 W25Q128JVS, U4 MCP2515-xSO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

Commit message: Ready first PCB
Parts:
- C10, C11, C12, C13, C14, C15, C16, C17, C5, C6, C7, C8, C9, R6, R7, R8: moved to B.Cu
- U1: moved to F.Cu
- moved C21 64.2 mm to (100.5, 100.5), turned to 90 degrees
- moved C20 63.5 mm to (101.0, 102.5), turned to 90 degrees
- moved C9 57.1 mm to (142.0, 73.5)
- moved C15 56.5 mm to (134.0, 70.0), turned to -90 degrees
- moved C16 56.5 mm to (136.0, 70.0), turned to -90 degrees
- moved C17 56.5 mm to (135.0, 70.0), turned to -90 degrees
- moved C13 56.1 mm to (142.0, 74.5)
- moved C8 56.1 mm to (140.0, 74.5)
- moved C12 55.0 mm to (142.0, 75.5)
- moved C7 55.0 mm to (140.0, 75.5)
- moved C11 54.1 mm to (142.0, 76.5)
- moved C6 54.1 mm to (140.0, 76.5)
- moved R5 53.4 mm to (136.0, 78.5), turned to 180 degrees
- moved C10 53.2 mm to (142.0, 77.5)
- moved C14 53.2 mm to (140.0, 77.5)
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Connections:
- J12 pad 7: +3.3V -> VBUS
- J12 pad 8: +3.3V -> VBUS
- J13 pad 7: +3.3V -> VBUS
- J13 pad 8: +3.3V -> VBUS
Routing:
- net GND: track 71.7 -> 293.9 mm, vias 4 -> 14
- net +3.3V: track 43.6 -> 173.3 mm, vias 1 -> 11
- net VBUS: track 12.6 -> 100.7 mm, vias 2 -> 4
- net GPIO19: track 0.00 -> 83.2 mm, vias 0 -> 4
- net GPIO20: track 0.00 -> 83.0 mm, vias 0 -> 4
- net GPIO18: track 0.00 -> 81.2 mm, vias 0 -> 4
- net GPIO16: track 0.00 -> 78.6 mm, vias 0 -> 2
- net GPIO17: track 0.00 -> 77.9 mm, vias 0 -> 2
- net Net-(U1-USB_DP): track 0.00 -> 54.6 mm, vias 0 -> 4
- net Net-(U1-USB_DM): track 0.00 -> 51.5 mm, vias 0 -> 2
- net CAN_H_IN: track 0.00 -> 50.3 mm, vias 0 -> 1
- net CAN_L_IN: track 0.00 -> 46.2 mm, vias 0 -> 1
- net QSPI_SS: track 0.00 -> 41.5 mm, vias 0 -> 1
- net GPIO15: track 0.00 -> 36.5 mm
- net GPIO14: track 0.00 -> 33.6 mm
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Other:
- outline, holes or cut-outs redrawn
